Commit message: Correct the CAD densities at source and rebuild the asset
The SolidWorks export had no materials assigned: 122 of 130 bodies at the
default 1000 kg/m^3, including all 16 that make up the three links. Patching
masses at runtime was not enough, because the error is not uniform within a
body -- steel hardware 7.85x up, PETG 0.48x down -- so the centres of mass and
inertias move too:

  l_com  link1  0.1079 -> 0.1659  (+53.6%)
         link2  0.1652 -> 0.2120  (+28.3%)
  mass   links  [0.1775,0.1003,0.0775] -> [0.1434,0.1063,0.0372]
  cart   0.4266 -> 0.6325;  cart:links 1.20 -> 2.20

A mass-only retrain was launched and then killed: it would have reached 100%
on a third robot that also does not exist. The correction is now applied to
bodies_raw.csv itself and the whole pipeline re-run (aggregate -> urdf -> usd),
with the original CSV and params preserved alongside. All 7 asset validation
checks pass and the rebuilt USD matches the corrected CAD to 1e-8 relative.

Classification is by part name and is reliable for the 16 link bodies, which
are individually identifiable. It is rougher for the 103 parts bucketed as
PETG elsewhere, some of which (the LiPo, for one) are certainly not printed
plastic. The base is static so this does not matter dynamically; the cart
carries more uncertainty than the link figures do. Nothing has been weighed --
hardware.yaml still has links_weighed_kg: null.

Co-Authored-By: Claude Opus 5 <noreply@anthropic.com>

File: assets/triple_pendulum/urdf/triple_pendulum.urdf (robot description, URDF)
Before this commit: robot triple_pendulum, 5 links, 4 joints
Links:
- link base_link: mass 7.34087816 -> 5.82490028
- link cart: mass 0.790531997 -> 0.996394613
- link link1: mass 0.177516137 -> 0.143393412
- link link2: mass 0.100255888 -> 0.106308493
- link link3: mass 0.0774675826 -> 0.0371844397
